File: Self-Balancing-Bot-Pid/PCBs/Motor Driver PCB/Motor Driver PCB.kicad_sch (KiCad schematic)
At the start: 23 parts, among them IC1 AS5600-ASOT, J1 Conn_01x08_Pin, U1 A4988SETTR-T

Commit message: Updated gitignore to ignore certain Kicad files. Ran ERC and DRC in Kicad, fixed any remaining issues, and now ready to route.
Parts:
- C6: footprint Capacitor_SMD:C_0603_1608Metric -> Capacitor_SMD:C_1210_3225Metric
Connections:
- net VDD: no longer IC1.1 (VDD5V)
- no-connect marks 2 -> 3
Changed lines of the file:
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@@
-	)
-	(junction
-		(at 215.9 105.41)
-		(diameter 0)
-		(color 0 0 0 0)
 	)
 	(junction
@@
 		(diameter 0)
 		(color 0 0 0 0)
+	)
+	(no_connect
+		(at 218.44 105.41)
 	)
 	(no_connect
@@
 	(wire
 		(pts
-			(xy 215.9 105.41) (xy 218.44 105.41)
-		)
-		(stroke
-			(width 0)
-			(type default)
-		)
-	)
-	(wire
-		(pts
 			(xy 152.4 100.33) (xy 176.53 100.33)
 		)
@@
 	(wire
 		(pts
-			(xy 215.9 105.41) (xy 215.9 107.95)
+			(xy 215.9 102.87) (xy 215.9 107.95)
 		)
 		(stroke
@@
 		(pts
 			(xy 104.14 110.49) (xy 104.14 90.17)
-		)
-		(stroke
-			(width 0)
-			(type default)
-		)
-	)
-	(wire
-		(pts
-			(xy 215.9 102.87) (xy 215.9 105.41)
 		)
 		(stroke
@@
 			)
 		)
-		(property "Footprint" "Capacitor_SMD:C_0603_1608Metric"
+		(property "Footprint" "Capacitor_SMD:C_1210_3225Metric"
 			(at 147.32 71.12 0)
 			(effects
